Commit message: hell nahn

File: ex01/robot.urdf (robot description, URDF)
Before this commit: robot robot_pylesos, 4 links, 3 joints
Links:
- link caster_wheel: mass 0.05 -> 0.1; geometry collision sphere radius=0.2; visual sphere radius=0.1
Joints:
- joint caster_joint: origin xyz=-0.12 0 -0.04 -> xyz=-0.15 0 0.0

File: ex02/robot.urdf.xacro (robot description, xacro)
@@ -1,8 +1,18 @@
 <?xml version="1.0"?>
-<robot xmlns:xacro="http://www.ros.org/wiki/xacro" name="pylesos">
-  <!-- === Материалы === -->
+<robot xmlns:xacro="http://ros.org/wiki/xacro" name="pylesos">
+  <!-- === Константы === -->
+  <xacro:property name="base_radius" value="0.18"/>
+  <xacro:property name="base_length" value="0.08"/>
+  <xacro:property name="wheel_radius" value="0.04"/>
+  <xacro:property name="wheel_length" value="0.02"/>
+  <xacro:property name="caster_radius" value="0.1"/>
+  <xacro:property name="caster_visual_z" value="0.08"/>
+  <xacro:property name="caster_collision_z" value="0.05"/>
+  <xacro:property name="wheel_offset_y" value="0.15"/>
+  <xacro:property name="caster_offset_x" value="-0.15"/>
   <xacro:property name="silver_color" value="0.7 0.7 0.7 1.0"/>
   <xacro:property name="black_color" value="0.05 0.05 0.05 1.0"/>
   <xacro:property name="darkgray_color" value="0.3 0.3 0.3 1.0"/>
+  <!-- === Материалы === -->
   <material name="silver">
     <color rgba="${silver_color}"/>
@@ -14,12 +24,6 @@
     <color rgba="${darkgray_color}"/>
   </material>
-  <!-- === Параметры робота === -->
-  <xacro:property name="base_radius" value="0.18"/>
-  <xacro:property name="base_length" value="0.08"/>
-  <xacro:property name="wheel_radius" value="0.04"/>
-  <xacro:property name="wheel_length" value="0.02"/>
-  <xacro:property name="caster_radius" value="0.025"/>
   <!-- === Макрос для колеса === -->
-  <xacro:macro name="wheel" params="name x y z material">
+  <xacro:macro name="wheel" params="name y material">
     <link name="${name}">
       <visual>
@@ -38,6 +42,5 @@
       <inertial>
         <mass value="0.1"/>
-        <inertia ixx="0.001" ixy="0.0" ixz="0.0"
-                 iyy="0.001" iyz="0.0" izz="0.001"/>
+        <inertia ixx="0.001" ixy="0" ixz="0" iyy="0.001" iyz="0" izz="0.001"/>
       </inertial>
     </link>
@@ -45,5 +48,5 @@
       <parent link="base_link"/>
       <child link="${name}"/>
-      <origin xyz="${x} ${y} ${z}" rpy="0 0 0"/>
+      <origin xyz="0 ${y} 0" rpy="0 0 0"/>
       <axis xyz="0 1 0"/>
     </joint>
@@ -66,11 +69,10 @@
     <inertial>
       <mass value="2.0"/>
-      <inertia ixx="0.02" ixy="0.0" ixz="0.0"
-               iyy="0.02" iyz="0.0" izz="0.03"/>
+      <inertia ixx="0.02" ixy="0" ixz="0" iyy="0.02" iyz="0" izz="0.03"/>
     </inertial>
   </link>
-  <!-- === Колёса === -->
-  <xacro:wheel name="left_wheel" x="0" y="0.15" z="0" material="black"/>
-  <xacro:wheel name="right_wheel" x="0" y="-0.15" z="0" material="black"/>
+  <!-- === Основные колеса === -->
+  <xacro:wheel name="left_wheel"  y="${wheel_offset_y}" material="black"/>
+  <xacro:wheel name="right_wheel" y="-${wheel_offset_y}" material="black"/>
   <!-- === Опорное колесо === -->
   <link name="caster_wheel">
@@ -79,17 +81,16 @@
         <sphere radius="${caster_radius}"/>
       </geometry>
-      <material name="darkgray"/>
-      <origin xyz="-0.12 0 -0.025"/>
+      <material name="silver"/>
+      <origin xyz="${caster_offset_x} 0 ${caster_visual_z}"/>
     </visual>
     <collision>
       <geometry>
-        <sphere radius="${caster_radius}"/>
+        <sphere radius="0.2"/>
       </geometry>
-      <origin xyz="-0.12 0 -0.025"/>
+      <origin xyz="${caster_offset_x} 0 ${caster_collision_z}"/>
     </collision>
     <inertial>
-      <mass value="0.05"/>
-      <inertia ixx="0.0002" ixy="0.0" ixz="0.0"
-               iyy="0.0002" iyz="0.0" izz="0.0002"/>
+      <mass value="0.1"/>
+      <inertia ixx="0.001" iyy="0.001" izz="0.001"/>
     </inertial>
   </link>
@@ -97,5 +98,5 @@
     <parent link="base_link"/>
     <child link="caster_wheel"/>
-    <origin xyz="-0.12 0 -0.04"/>
+    <origin xyz="${caster_offset_x} 0 0.0"/>
   </joint>
 </robot>

Commit message: lab 5

File: ex01/robot.urdf (robot description, URDF)
Before this commit: robot pylesos, 4 links, 3 joints
Links:
- link caster_wheel: mass 0.1 -> 0.05; geometry collision cylinder length=0.015 radius=0.025; visual cylinder length=0.015 radius=0.025
Joints:
- joint caster_joint: axis (none) -> 0 0 1; origin xyz=-0.15 0 0.0 -> xyz=-0.15 0 0.01; type fixed -> continuous

File: ex03/urdf/robot.urdf.xacro (robot description, xacro)
@@ -77,19 +77,19 @@
   <link name="caster_wheel">
     <visual>
-      <origin xyz="0 0 0" rpy="1.5708 0 0"/>
+      <origin xyz="0 0 0" rpy="0 0 0"/>
       <geometry>
-        <cylinder radius="${caster_radius}" length="0.015"/>
+        <sphere radius="${caster_radius}"/>
       </geometry>
       <material name="darkgray"/>
     </visual>
     <collision>
-      <origin xyz="0 0 0" rpy="1.5708 0 0"/>
+      <origin xyz="0 0 0" rpy="0 0 0"/>
       <geometry>
-        <cylinder radius="${caster_radius}" length="0.015"/>
+        <sphere radius="${caster_radius}"/>
       </geometry>
     </collision>
     <inertial>
       <mass value="0.05"/>
-      <inertia ixx="0.0002" ixy="0" ixz="0" iyy="0.0002" iyz="0" izz="0.0002"/>
+      <inertia ixx="0.00002" ixy="0" ixz="0" iyy="0.00002" iyz="0" izz="0.00002"/>
     </inertial>
   </link>
